File: electrical/Electrical_Diagram/Electrical_Diagram.kicad_sch (KiCad schematic)
At the start: 25 parts

Commit message: updated electrical
Parts:
- added A1: Arduino_UNO_R3, Module:Arduino_UNO_R3, symbol MCU_Module:Arduino_UNO_R3
- added BMS1: ~, symbol [TT]Library:bms
Connections:
- net at BT1.2 (-), BT12.2 (-), BT15.2 (-)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: now also BMS1. (VBUS)
- net at BT10.1 (+), BT13.1 (+), BT16.1 (+)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: now also BMS1. (VBUS)
- net at BT2.1 (+), BT3.2 (-): now also BMS1. (VBUS)
- net at BT1.1 (+), BT2.2 (-): now also BMS1. (VBUS)
- net GND: now reaches Pi_1. (VBUS)
- net GND: now also BMS1. (VBUS)
- net at Pi_1.1 (VBUS1): now also A1. (USB_VBUS)
- net at Pi_1.2 (D1-): now also A1. (USB_VBUS)
- net at Pi_1.3 (D1+): now also A1. (USB_VBUS)
- net at Pi_1.8 (GND2): now also A1. (USB_VBUS)
- new net +5V: Pi_1. (VBUS)
- new net VBUS: BMS1. (VBUS)
Other:
- moved on the sheet: BT1, BT10, BT11, BT12, BT13, BT14, BT15, BT16, BT17, BT18, BT19, BT2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
