File: electrical/Electrical_Diagram/Electrical_Diagram.kicad_sch (KiCad schematic)
At the start: 28 parts

Commit message: reupdated kicad
Parts:
- added CAM1: ~, symbol [TT]Library:CAMERA
- added M1, M2: Motor_DC, symbol Motor:Motor_DC
- renumbered U1 to MOTORSHEILD
Connections:
- net GND: now also A1.29 (GND), A1.6 (GND), A1.7 (GND), MOTORSHEILD.29 (GND), MOTORSHEILD.6 (GND), MOTORSHEILD.7 (GND)
- net VBUS: now also MOTORSHEILD.8 (VIN)
- net at BT23.2 (-), BT24.1 (+): now also BMS1. (VBUS), BT1.1 (+), BT11.2 (-), BT12.1 (+), BT14.2 (-), BT15.1 (+), BT17.2 (-), BT18.1 (+), BT2.2 (-), BT20.2 (-), BT21.1 (+), BT5.2 (-), BT6.1 (+), BT8.2 (-), BT9.1 (+)
- net at BT22.2 (-), BT23.1 (+): now also BMS1. (VBUS), BT10.2 (-), BT11.1 (+), BT13.2 (-), BT14.1 (+), BT16.2 (-), BT17.1 (+), BT19.2 (-), BT2.1 (+), BT20.1 (+), BT3.2 (-), BT4.2 (-), BT5.1 (+), BT7.2 (-), BT8.1 (+)
- net A1: now reaches MOTORSHEILD.10 (A1)
- net A1: now also A1.10 (A1)
- net A2: now reaches MOTORSHEILD.11 (A2)
- net A2: now also A1.11 (A2)
- net A3: now reaches MOTORSHEILD.12 (A3)
- net A3: now also A1.12 (A3)
- net A4: now reaches MOTORSHEILD.13 (SDA/A4)
- net A4: now also A1.13 (SDA/A4), A1.31 (SDA/A4), MOTORSHEILD.31 (SDA/A4)
- net A5: now reaches MOTORSHEILD.14 (SCL/A5)
- net A5: now also A1.14 (SCL/A5), A1.32 (SCL/A5), MOTORSHEILD.32 (SCL/A5)
- net RX: now reaches MOTORSHEILD.15 (D0/RX)
- net RX: now also A1.15 (D0/RX)
- net TX: now reaches MOTORSHEILD.16 (D1/TX)
- net TX: now also A1.16 (D1/TX)
- net D2: now reaches MOTORSHEILD.17 (D2)
- net D2: now also A1.17 (D2)
- net D3: now reaches MOTORSHEILD.18 (D3)
- net D3: now also A1.18 (D3)
- net D4: now reaches MOTORSHEILD.19 (D4)
- net D4: now also A1.19 (D4)
- net D5: now reaches MOTORSHEILD.20 (D5)
- net D5: now also A1.20 (D5)
- net D6: now reaches MOTORSHEILD.21 (D6)
- net D6: now also A1.21 (D6)
- net D7: now reaches MOTORSHEILD.22 (D7)
- net D7: now also A1.22 (D7)
- net D8: now reaches MOTORSHEILD.23 (D8)
- net D8: now also A1.23 (D8)
- net D9: now reaches MOTORSHEILD.24 (D9)
- net D9: now also A1.24 (D9)
- net D10: now reaches MOTORSHEILD.25 (D10)
- net D10: now also A1.25 (D10)
- net D11: now reaches MOTORSHEILD.26 (D11)
- net D11: now also A1.26 (D11)
- net D12: now reaches MOTORSHEILD.27 (D12)
- net D12: now also A1.27 (D12)
- net D13: now reaches MOTORSHEILD.28 (D13)
- net D13: now also A1.28 (D13)
- net A0: now reaches MOTORSHEILD.9 (A0)
- net A0: now also A1.9 (A0)
- net UNO_VBUS: now reaches Pi_1.1 (VBUS1)
- net UNO_VBUS: now also A1. (USB_VBUS)
- net UNO_D-: now reaches Pi_1.2 (D1-)
- net UNO_D-: now also A1. (USB_VBUS)
- net UNO_D+: now reaches Pi_1.3 (D1+)
- net UNO_D+: now also A1. (USB_VBUS)
- net UNO_USB_GND: now reaches Pi_1.4 (GND1)
- net UNO_USB_GND: now also A1. (USB_VBUS)
- new net: CAM1. (USB__VBUS), Pi_1.1 (VBUS1)
- new net: CAM1. (USB__VBUS), Pi_1.2 (D1-)
- new net: CAM1. (USB__VBUS), Pi_1.3 (D1+)
- new net: CAM1. (USB__VBUS), Pi_1.4 (GND1)
- new net: M2.1 (+), MOTORSHEILD. (M4B)
- new net: M2.2 (-), MOTORSHEILD. (M4B)
- new net: M1.1 (+), MOTORSHEILD. (M4B)
- new net: M1.2 (-), MOTORSHEILD. (M4B)
- now unconnected: Pi_1.8 (GND2)
- no-connect marks 0 -> 12
Other:
- moved on the sheet: A1, Reference: MOTORSHEILD

Commit message: finished rev 1 of electrical
Parts:
- added Encoder1, Encoder2: ~, symbol [TT]Library:RotaryEncoder
- added SCREEN1: ~, symbol [TT]Library:SCREEN
- added SR1, SR2, SR3: ~, symbol [TT]Library:HC-SR04
Connections:
- net A0: now also Encoder2. (VIN)
- net A1: now also Encoder2. (VIN)
- net A2: now also Encoder1. (VIN)
- net A4: now also Encoder1. (VIN)
- net D11: now also SR1. (VIN)
- net D12: now also SR2. (VIN)
- net D13: now also SR3. (VIN)
- net D2: now also SR1. (VIN), SR2. (VIN), SR3. (VIN)
- net GND: no longer A1.29 (GND), A1.6 (GND), A1.7 (GND), MOTORSHEILD.29 (GND), MOTORSHEILD.6 (GND), MOTORSHEILD.7 (GND)
- net at CAM1. (USB__VBUS): now also Pi_1.4 (GND1); no longer Pi_1.1 (VBUS1)
- net at A1.5 (+5V): now also SR1. (VIN), SR2. (VIN), SR3. (VIN)
- new net: CAM1. (USB__VBUS), Pi_1.1 (VBUS1)
- new net: CAM1. (USB__VBUS), Pi_1.2 (D1-)
- new net: CAM1. (USB__VBUS), Pi_1.3 (D1+)
- new net: Pi_1. (VBUS), SCREEN1. (VBUS)
- new net: Pi_1.5 (VBUS2), SCREEN1. (VBUS)
- new net: Pi_1.6 (D2-), SCREEN1. (VBUS)
- new net: Pi_1.7 (D2+), SCREEN1. (VBUS)
- new net: Pi_1.8 (GND2), SCREEN1. (VBUS)
- new net 5V: Encoder1. (VIN), Encoder2. (VIN), MOTORSHEILD.7 (+5V)
- new net GND1: A1.29 (GND), A1.6 (GND), A1.7 (GND), Encoder1. (VIN), Encoder2. (VIN), MOTORSHEILD.29 (GND), MOTORSHEILD.6 (GND), SR1. (VIN), SR2. (VIN), SR3. (VIN)
- no-connect marks 12 -> 18
Other:
- note added: "NOTE: D3 TO D10 UNUSABLE (USED TO COMMUNICATE MOTOR DIRECTION AND SPEED TO MOTOR SHIELD)"
- note added: "NOTE: HDMI WIRE REPRESENTS HDMI BUS"
- company: (none) -> [TT] ZETA BETA
- title: (none) -> ELECTRICAL DIAGRAM
- moved on the sheet: A1, CAM1, M1, M2, MOTORSHEILD
